Commit message: Fixed robot state publisher and updated test joint state publisher

File: python_lcm_msgs/assets/devkit_base_descr.urdf (robot description, URDF)
Before this commit: robot devkit_base_descr, 15 links, 14 joints
Links:
- added link pan_tilt_base; collision mesh filename=package://dim_cpp/meshes/devkit_base/pan_tilt_base_collisio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 scale=1 1 1; visual mesh filename=package://dim_cpp/meshes/devkit_base/pan_tilt_base_collisio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 scale=1 1 1
- added link pan_tilt_head; collision mesh filename=package://dim_cpp/meshes/devkit_base/pan_tilt_head_collisio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 scale=1 1 1; visual mesh filename=package://dim_cpp/meshes/devkit_base/pan_tilt_head_collisio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 scale=1 1 1
- added link pan_tilt_pan; collision mesh filename=package://dim_cpp/meshes/devkit_base/pan_tilt_pan_collision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 scale=1 1 1; visual mesh filename=package://dim_cpp/meshes/devkit_base/pan_tilt_pan_collision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 scale=1 1 1
- link base_link: mass None -> 1.02
- link devkit_base_link: mass None -> 45
- link gripper_base: mass None -> 0.45
- link link1: mass None -> 0.71
- link link2: mass None -> 1.17
- link link3: mass None -> 0.5
- link link4: mass None -> 0.38
- link link5: mass None -> 0.383
- link link6: mass None -> 0.00699089613564366
- link link7: mass None -> 0.025
- link link8: mass None -> 0.025
- link pillar_platform: mass None -> 1.5
- link piper_angled_mount: mass None -> 1.5
Joints:
- added joint pan_tilt_base_joint: type fixed, parent devkit_base_link, child pan_tilt_base, origin xyz=0 0 0 rpy=0 0 0
- added joint pan_tilt_head_joint: type revolute, parent pan_tilt_pan, child pan_tilt_head, origin xyz=0 0 1.6465 rpy=0 0 0, axis 1 0 0, limit lower=-1.57 upper=1.57 effort=100 velocity=1
- added joint pan_tilt_pan_joint: type revolute, parent pan_tilt_base, child pan_tilt_pan, origin xyz=0 .1325 0 rpy=0 0 0, axis 0 0 1, limit lower=-3.14 upper=3.14 effort=100 velocity=1
