Commit message: Added obj files and modified assets

File: assets/devkit_base_descr.urdf (robot description, URDF)
Before this commit: robot devkit_base_descr, 19 links, 18 joints
Links:
- link base_link: geometry collision mesh filename=dim_cpp/piper_description/meshes/base_link.obj; visual mesh filename=dim_cpp/piper_description/meshes/base_link.obj
- link devkit_base_link: geometry collision mesh filename=dim_cpp/meshes/devkit_base/devkit_base_wheels_collision.obj scale=1 1 1; visual mesh filename=dim_cpp/meshes/devkit_base/devkit_base_wheels_collision.obj scale=1 1 1
- link gripper_base: geometry collision mesh filename=dim_cpp/piper_description/meshes/gripper_base.obj; visual mesh filename=dim_cpp/piper_description/meshes/gripper_base.obj
- link link1: geometry collision mesh filename=dim_cpp/piper_description/meshes/link1.obj; visual mesh filename=dim_cpp/piper_description/meshes/link1.obj
- link link2: geometry collision mesh filename=dim_cpp/piper_description/meshes/link2.obj; visual mesh filename=dim_cpp/piper_description/meshes/link2.obj
- link link3: geometry collision mesh filename=dim_cpp/piper_description/meshes/link3.obj; visual mesh filename=dim_cpp/piper_description/meshes/link3.obj
- link link4: geometry collision mesh filename=dim_cpp/piper_description/meshes/link4.obj; visual mesh filename=dim_cpp/piper_description/meshes/link4.obj
- link link5: geometry collision mesh filename=dim_cpp/piper_description/meshes/link5.obj; visual mesh filename=dim_cpp/piper_description/meshes/link5.obj
- link link6: geometry collision mesh filename=dim_cpp/piper_description/meshes/link6.obj; visual mesh filename=dim_cpp/piper_description/meshes/link6.obj
- link link7: geometry collision mesh filename=dim_cpp/piper_description/meshes/link7.obj; visual mesh filename=dim_cpp/piper_description/meshes/link7.obj
- link link8: geometry collision mesh filename=dim_cpp/piper_description/meshes/link8.obj; visual mesh filename=dim_cpp/piper_description/meshes/link8.obj
- link pan_tilt_base: geometry collision mesh filename=dim_cpp/meshes/devkit_base/pan_tilt_base_collision.obj scale=1 1 1; visual mesh filename=dim_cpp/meshes/devkit_base/pan_tilt_base_collision.obj scale=1 1 1
- link pan_tilt_head: geometry collision mesh filename=dim_cpp/meshes/devkit_base/pan_tilt_head_collision.obj scale=1 1 1; visual mesh filename=dim_cpp/meshes/devkit_base/pan_tilt_head_collision.obj scale=1 1 1
- link pan_tilt_pan: geometry collision mesh filename=dim_cpp/meshes/devkit_base/pan_tilt_pan_collision.obj scale=1 1 1; visual mesh filename=dim_cpp/meshes/devkit_base/pan_tilt_pan_collision.obj scale=1 1 1
- link pillar_platform: geometry collision mesh filename=dim_cpp/meshes/devkit_base/pillar_platform_collision.obj scale=1 1 1; visual mesh filename=dim_cpp/meshes/devkit_base/pillar_platform_collision.obj scale=1 1 1
- link piper_angled_mount: geometry collision mesh filename=dim_cpp/meshes/devkit_base/piper_angled_mount_collision.obj scale=1 1 1; visual mesh filename=dim_cpp/meshes/devkit_base/piper_angled_mount_collision.obj scale=1 1 1
