Commit message: URDF with zed and ft min driver

File: assets/dim_cpp/urdf/xarm6_openft_gripper.urdf (robot description, URDF)
Before this commit: robot xarm_openft_gripper, 19 links, 18 joints
Links:
- added link zed_camera_center; collision mesh filename=package://dim_cpp/meshes/zedm.stl; visual mesh filename=package://dim_cpp/meshes/zedm.stl
- added link zed_camera_link
- added link zed_left_camera_frame
- added link zed_left_camera_optical_frame
- added link zed_right_camera_frame
- added link zed_right_camera_optical_frame
Joints:
- added joint zed_camera_center_joint: type fixed, parent zed_camera_link, child zed_camera_center, origin xyz=0 0 0.01325 rpy=0 0.0 0
- added joint zed_fixed_joint: type fixed, parent link_openft, child zed_camera_link, origin xyz=0 .08605 .02325 rpy=0 -1.5707 -1.5707
- added joint zed_left_camera_joint: type fixed, parent zed_camera_center, child zed_left_camera_frame, origin xyz=0.0 0.0315 0 rpy=0 0 0
- added joint zed_left_camera_optical_joint: type fixed, parent zed_left_camera_frame, child zed_left_camera_optical_frame, origin xyz=0 0 0 rpy=-1.5707963267948966 0.0 -1.5707963267948966
- added joint zed_right_camera_joint: type fixed, parent zed_camera_center, child zed_right_camera_frame, origin xyz=0.0 -0.0315 0 rpy=0 0 0
- added joint zed_right_camera_optical_joint: type fixed, parent zed_right_camera_frame, child zed_right_camera_optical_frame, origin xyz=0 0 0 rpy=-1.5707963267948966 0.0 -1.5707963267948966
- joint gripper_fix: origin xyz=0 0 0.015 rpy=0 0 -1.570796 -> xyz=0 0 0.025 rpy=0 0 -1.570796

File: assets/xarm6_openft_gripper.urdf (robot description, URDF)
Before this commit: robot xarm_openft_gripper, 19 links, 18 joints
Links:
- added link zed_camera_center; collision mesh filename=dim_cpp/meshes/zedm.obj; visual mesh filename=dim_cpp/meshes/zedm.obj
- added link zed_camera_link
- added link zed_left_camera_frame
- added link zed_left_camera_optical_frame
- added link zed_right_camera_frame
- added link zed_right_camera_optical_frame
Joints:
- added joint zed_camera_center_joint: type fixed, parent zed_camera_link, child zed_camera_center, origin xyz=0 0 0.01325 rpy=0 0.0 0
- added joint zed_fixed_joint: type fixed, parent link_openft, child zed_camera_link, origin xyz=0 .08605 .02325 rpy=0 -1.5707 -1.5707
- added joint zed_left_camera_joint: type fixed, parent zed_camera_center, child zed_left_camera_frame, origin xyz=0.0 0.0315 0 rpy=0 0 0
- added joint zed_left_camera_optical_joint: type fixed, parent zed_left_camera_frame, child zed_left_camera_optical_frame, origin xyz=0 0 0 rpy=-1.5707963267948966 0.0 -1.5707963267948966
- added joint zed_right_camera_joint: type fixed, parent zed_camera_center, child zed_right_camera_frame, origin xyz=0.0 -0.0315 0 rpy=0 0 0
- added joint zed_right_camera_optical_joint: type fixed, parent zed_right_camera_frame, child zed_right_camera_optical_frame, origin xyz=0 0 0 rpy=-1.5707963267948966 0.0 -1.5707963267948966
- joint gripper_fix: origin xyz=0 0 0.015 rpy=0 0 -1.570796 -> xyz=0 0 0.025 rpy=0 0 -1.570796
